File: pcb/SolarMeshtasticNodeMini.kicad_pcb (KiCad board)
At the start: 4 copper layers, 33 x 47 mm, 31 parts, among them J2 Conn_01x02_Socket, J3 Conn_01x04_Socket, J4 Conn_01x02_Pin, J5 Conn_01x04_Socket, SW1 SSSS811101, SW2 SW_Push, U1 BQ25185, U2 HT-CT62, U3 HE9073A30MR, U4 APX803L05-32SA-7, U9 SS26_C5350986

Commit message: pcb: optimize 3v3 and gnd rails a bit
Routing:
- net GND: vias 117 -> 119
Other:
- board text added: "Boot: A -> Application B -> Bootloader ISET: 300Ohm -> 1A ILM: 100kOhm -> 4.1V@1100mA 13kOhm -> 4.2V@1100mA"
- board text removed: "Boot: GPIO9 = 1: SW GPIO9 = 0: BL ISET: 300Ohm -> 1A ILM: 100kOhm -> 4.1V@1100mA 13kOhm -> 4.2V@1100mA"

Commit message: pcb, sch: add load switch to control entire 3.3V rail
Until now only the ESP32 was disabled if the voltage drops due to
discharge. This might cause the sensors to slip into a slow brown-out.
Parts:
- added C9: 1uF, Capacitor_SMD:C_0805_2012Metric_Pad1.18x1.45mm_HandSolder, F.Cu at (220.6, 66.6)
- added U5: TPS22917DBV, Package_TO_SOT_SMD:SOT-23-6, F.Cu at (217.5, 66.6)
- moved U9 2.81 mm to (218.2, 60.0), turned to 0 degrees
Connections:
- C4 pad 1: +3V3 -> /VOUT
- R10 pad 2: /ESP32_ENABLE -> /nReset
- R5 pad 2: /ESP32_ENABLE -> /nReset
- U2 pad 11: /ESP32_ENABLE -> +3V3
- U3 pad 3: +3V3 -> /VOUT
- U4 pad 2: /ESP32_ENABLE -> /nReset
Routing:
- net /ESP32_ENABLE: track 26.5 -> 0.00 mm, vias 3 -> 0
- net /nReset: track 0.00 -> 19.8 mm
- net /VOUT: track 0.00 -> 5.83 mm
- net /VBUS: track 25.3 -> 30.4 mm
- net GND: track 31.1 -> 32.8 mm, vias 119 -> 124
- net Net-(J3-Pin_2): track 11.3 -> 10.1 mm
- net +3V3: track 16.1 -> 16.0 mm, vias 7 -> 9
Other:
- board text added: "v0.0.3"
- board text removed: "v0.0.2"

Commit message: pcb, sch: replace reset ic with TI TPS3890 to get rid of bouncing behaviour
Parts:
- removed C7: 1uF, Capacitor_SMD:C_1206_3216Metric_Pad1.33x1.80mm_HandSolder
- removed R10: 100k, Resistor_SMD:R_0805_2012Metric_Pad1.20x1.40mm_HandSolder
- removed R5: 470, Resistor_SMD:R_0805_2012Metric_Pad1.20x1.40mm_HandSolder
- removed SW2: SW_Push, footprints:SMA_L4.3-W2.6-LS5.1-RD
- removed U4: APX803L05-32SA-7, footprints:SOT23-3
- removed U9: SS26_C5350986, footprints:SMA_L4.3-W2.6-LS5.1-RD
- added C10: 100nF, Capacitor_SMD:C_0805_2012Metric_Pad1.18x1.45mm_HandSolder, F.Cu at (219.7, 62.1)
- added C11: C, Capacitor_SMD:C_0805_2012Metric_Pad1.18x1.45mm_HandSolder, F.Cu at (223.5, 61.8)
- added R7: 1M, Resistor_SMD:R_0805_2012Metric_Pad1.20x1.40mm_HandSolder, F.Cu at (223.5, 59.8)
- added R8: 470, Resistor_SMD:R_0805_2012Metric_Pad1.20x1.40mm_HandSolder, F.Cu at (223.4, 57.7)
- added SW3: SW_Push, footprints:SMA_L4.3-W2.6-LS5.1-RD, F.Cu at (231.3, 58.1)
- added U6: ~, Package_SON:WSON-6-1EP_2x2mm_P0.65mm_EP1x1.6mm, F.Cu at (220.3, 59.9)
Connections:
- J3 pad 2: Net-(J3-Pin_2) -> +3V3
Routing:
- net /VBUS: track 30.4 -> 4.88 mm, vias 1 -> 0
- net Net-(J3-Pin_2): track 10.1 -> 0.00 mm
- net /VLOAD: track 20.2 -> 30.1 mm
- net Net-(R8-Pad1): track 0.00 -> 4.33 mm
- net Net-(U6-CT): track 0.00 -> 2.51 mm
- net /nReset: track 19.8 -> 22.3 mm
- net Net-(R5-Pad1): track 2.41 -> 0.00 mm
- net GND: track 32.8 -> 32.6 mm, vias 124 -> 128
Other:
- board text added: "RST"
- board text added: "v0.0.x"
- board text removed: "v0.0.3"
