File: pcb/SolarMeshtasticNodeMini.kicad_pcb (KiCad board)
At the start: 4 copper layers, 33 x 47 mm, 34 parts, among them J2 Conn_01x02_Socket, J3 Conn_01x04_Socket, J4 Conn_01x02_Pin, J5 Conn_01x04_Socket, SW1 SSSS811101, SW2 SW_Push, U1 BQ25185, U2 HT-CT62, U3 HE9073A30MR, U4 APX803L05-32SA-7, U5 TPS22917DBV, U9 SS26_C5350986

Commit message: pcb, sch: add TVS protection to inputs
Parts:
- added D1: SMAJ5.0A, Diode_SMD:D_SMA, F.Cu at (222.3, 72.5)
- added D3: SMAJ15A, Diode_SMD:D_SMA, F.Cu at (236.6, 66.4)
- moved C10 7.42 mm to (214.6, 63.8), turned to 0 degrees
- moved J2 4.44 mm to (241.8, 67.8)
- moved J4 3.22 mm to (217.9, 72.3)
Routing:
- net /VLIPO: track 11.9 -> 17.1 mm
- net /VBUS: track 30.4 -> 34.3 mm, vias 1 -> 2
- net GND: track 33.7 -> 36.0 mm, vias 126 -> 132
- net /nReset: track 25.9 -> 24.3 mm
Other:
- board text added: "v1.0.0"
- board text removed: "v0.1.0"

Commit message: pcb, sch: we are using 3V0 everywhere. Also fix misleading comment in schematic regarding SYS voltage within the voltage divier
Connections:
- net +3V3 renamed +3V0
Other:
- board text added: "3V0"
- board text removed: "3V3"

Commit message: pcb, sch: add 1nF C to power switch to limit inrush
Parts:
- added C11: 1nF, Capacitor_SMD:C_0805_2012Metric_Pad1.18x1.45mm_HandSolder, F.Cu at (214.4, 66.8)
Connections:
- U5 pad 4: unconnected-(U5-CT-Pad4) -> Net-(U5-CT)
Routing:
- net /VOUT: track 5.69 -> 11.7 mm
- net Net-(U5-CT): track 0.00 -> 2.09 mm
- net GND: track 36.0 -> 36.4 mm, vias 132 -> 140

Commit message: pcb, sch: remove tvs from VBat to avoid draining
Parts:
- removed D1: SMAJ5.0A, Diode_SMD:D_SMA
- D3: value SMAJ15A -> SMAJ14A
- moved J4 2.39 mm to (220.3, 72.0)
Routing:
- net /VLIPO: track 17.1 -> 12.6 mm
- net GND: track 36.4 -> 34.6 mm
- net /VBUS: track 34.3 -> 33.5 mm

Commit message: pcb, sch: GPIO is the NSS of the SX1262. Do not pull high.
Connections:
- U2 pad 16: +3V0 -> unconnected-(U2-GPIO8-Pad16)
Routing:
- net unconnected-(U2-GPIO8-Pad16): track 0.00 -> 1.74 mm, vias 0 -> 1
- net +3V0: track 16.7 -> 14.9 mm, vias 9 -> 8
Changed lines of the file:
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@@
 		)
 		(pad_to_mask_clearance 0)
-		(solder_mask_min_width 0.1016)
 		(allow_soldermask_bridges_in_footprints no)
 		(tenting
@@
 			(layers "F.Cu" "F.Mask" "F.Paste")
 			(roundrect_rratio 0.25)
-			(net "+3V0")
+			(net "unconnected-(U2-GPIO8-Pad16)")
 			(pinfunction "GPIO8_16")
 			(pintype "bidirectional")
@@
 	)
 	(segment
-		(start 224.6 45.2)
-		(end 223.91 45.89)
-		(width 0.6)
-		(layer "F.Cu")
-		(net "+3V0")
-	)
-	(segment
 		(start 223.722934 36.7875)
 		(end 223.722934 38.98)
@@
 	)
 	(segment
-		(start 223.91 45.89)
-		(end 223.15 45.89)
-		(width 0.6)
-		(layer "F.Cu")
-		(net "+3V0")
-	)
-	(segment
 		(start 230.08 33.76)
 		(end 230.08 34.77)
@@
 	)
 	(via
-		(at 224.6 45.2)
-		(size 0.6858)
-		(drill 0.3302)
-		(layers "F.Cu" "B.Cu")
-		(net "+3V0")
-	)
-	(via
 		(at 228.07 33.81)
 		(size 0.6)
@@
 		(net "/ESP32_BOOTLOADER_MODE_1")
 	)
+	(segment
+		(start 224.6 45.2)
+		(end 223.91 45.89)
+		(width 0.6)
+		(layer "F.Cu")
+		(net "unconnected-(U2-GPIO8-Pad16)")
+	)
+	(segment
+		(start 223.91 45.89)
+		(end 223.15 45.89)
+		(width 0.6)
+		(layer "F.Cu")
+		(net "unconnected-(U2-GPIO8-Pad16)")
+	)
+	(via
+		(at 224.6 45.2)
+		(size 0.6858)
+		(drill 0.3302)
+		(layers "F.Cu" "B.Cu")
+		(net "unconnected-(U2-GPIO8-Pad16)")
+	)
 	(zone
