File: pcb/SolarMeshtasticNodeMini.kicad_sch (KiCad schematic)
At the start: 33 parts, among them J2 Conn_01x02_Socket, J3 Conn_01x04_Socket, J4 Conn_01x02_Pin, J5 Conn_01x04_Socket, SW1 SSSS811101, SW2 SW_Push, U1 BQ25185, U2 HT-CT62, U3 HE9073A30MR, U4 APX803L05-32SA-7, U5 TPS22917DBV, U9 SS26_C5350986

Commit message: pcb, sch: move nRST pull-up R10 from +3V3 to /VOUT
Connections:
- net +3V3: no longer R10.1
- net VLOAD: now also R10.1

Commit message: pcb, sch: add 1M:1M to the voltage divider
Parts:
- R13, R14: value R -> 1M
Changed lines of the file:
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@@
 			)
 		)
-		(property "Value" "R"
+		(property "Value" "1M"
 			(at 293.37 46.9899 0)
 			(show_name no)
@@
 			)
 		)
-		(property "Value" "R"
+		(property "Value" "1M"
 			(at 293.37 35.5599 0)
 			(show_name no)
