File: pcb/SolarMeshtasticNodeMini.kicad_sch (KiCad schematic)
At the start: 33 parts, among them J2 Conn_01x02_Socket, J3 Conn_01x04_Socket, J4 Conn_01x02_Pin, J5 Conn_01x04_Socket, SW1 SSSS811101, SW2 SW_Push, U1 BQ25185, U2 HT-CT62, U3 HE9073A30MR, U4 APX803L05-32SA-7, U5 TPS22917DBV, U9 SS26_C5350986

Commit message: pcb, sch: pull GPIO8 to high - otherwise uart bootloader mode might be unreliable
Connections:
- net +3V3: now also U2.16 (GPIO8)
- no-connect marks 15 -> 14
Changed lines of the file:
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@@
-	)
-	(no_connect
-		(at 232.41 80.01)
 	)
 	(no_connect
@@
 	(wire
 		(pts
+			(xy 232.41 80.01) (xy 234.95 80.01)
+		)
+		(stroke
+			(width 0)
+			(type default)
+		)
+	)
+	(wire
+		(pts
 			(xy 78.74 45.72) (xy 85.09 45.72)
 		)
@@
 		(effects
 			(font
+				(size 1.27 1.27)
+			)
+			(justify left bottom)
+		)
+	)
+	(label "+3V3"
+		(at 234.95 80.01 0)
+		(effects
+			(font

Commit message: pcb, sch: add 10uF to nReset to slow down resets from 50ms to 0.4s
Parts:
- added C10: 1uF, Capacitor_SMD:C_0805_2012Metric_Pad1.18x1.45mm_HandSolder, symbol Device:C
Connections:
- net GND: now also C10.1
- net nReset: now also C10.2
Other:
- note added: "Adds roughly ~0.4s to RST"
Changed lines of the file:
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@@
 		)
 	)
+	(text "Adds roughly\n~0.4s to RST"
+		(exclude_from_sim no)
+		(at 176.022 232.41 0)
+		(effects
+			(font
+				(size 1.27 1.27)
+			)
+		)
+	)
 	(text "USART"
 		(exclude_from_sim no)
@@
 	)
 	(junction
+		(at 166.37 218.44)
+		(diameter 0)
+		(color 0 0 0 0)
+	)
+	(junction
 		(at 290.83 41.91)
 		(diameter 0)
@@
 	(wire
 		(pts
+			(xy 166.37 226.06) (xy 166.37 228.6)
+		)
+		(stroke
+			(width 0)
+			(type default)
+		)
+	)
+	(wire
+		(pts
 			(xy 189.23 157.48) (xy 194.31 157.48)
 		)
@@
 	(wire
 		(pts
-			(xy 156.21 218.44) (xy 162.56 218.44)
+			(xy 156.21 218.44) (xy 166.37 218.44)
 		)
 		(stroke
@@
 	(wire
 		(pts
+			(xy 166.37 218.44) (xy 176.53 218.44)
+		)
+		(stroke
+			(width 0)
+			(type default)
+		)
+	)
+	(wire
+		(pts
 			(xy 83.82 130.81) (xy 83.82 132.08)
 		)
@@
 	)
 	(label "nReset"
-		(at 162.56 218.44 0)
+		(at 176.53 218.44 0)
 		(effects
 			(font
@@
 		(in_pos_files yes)
 		(dnp no)
-		(fields_autoplaced yes)
 		(property "Reference" "U5"
 			(at 204.47 144.78 0)
@@
 		)
 		(property "Value" "TPS22917DBV"
-			(at 204.47 147.32 0)
+			(at 205.74 148.59 0)
 			(show_name no)
 			(do_not_autoplace no)
@@
 	(symbol
 		(lib_id "Device:C")
+		(at 166.37 222.25 180)
+		(unit 1)
+		(body_style 1)
+		(exclude_from_sim no)
+		(in_bom yes)
+		(on_board yes)
+		(in_pos_files yes)
+		(dnp no)
+		(fields_autoplaced yes)
+		(property "Reference" "C10"
+			(at 170.18 220.9799 0)
+			(show_name no)
+			(do_not_autoplace no)
+			(effects
+				(font
+					(size 1.27 1.27)
+				)
+				(justify right)
+			)
+		)
+		(property "Value" "1uF"
+			(at 170.18 223.5199 0)
+			(show_name no)
+			(do_not_autoplace no)
+			(effects
+				(font
+					(size 1.27 1.27)
+				)
+				(justify right)
+			)
+		)
+		(property "Footprint" "Capacitor_SMD:C_0805_2012Metric_Pad1.18x1.45mm_HandSolder"
+			(at 165.4048 218.44 0)
+			(hide yes)
+			(show_name no)
+			(do_not_autoplace no)
+			(effects
+				(font
+					(size 1.27 1.27)
+				)
+			)
+		)
+		(property "Datasheet" ""
+			(at 166.37 222.25 0)
+			(hide yes)
+			(show_name no)
+			(do_not_autoplace no)
+			(effects
+				(font
+					(size 1.27 1.27)
+				)
+			)
+		)
+		(property "Description" "Unpolarized capacitor"
+			(at 166.37 222.25 0)
+			(hide yes)
+			(show_name no)
+			(do_not_autoplace no)
+			(effects
+				(font
+					(size 1.27 1.27)
+				)
+			)
+		)
+		(pin "2"
+		)
+		(pin "1"
+		)
+		(instances
+			(project "SolarMeshtasticNodeMini"
+				(path "/256f162e-4f54-42b3-a315-b65231ce36a5"
+					(reference "C10")
+					(unit 1)
+				)
+			)
+		)
+	)
+	(symbol
+		(lib_id "Device:C")
 		(at 127 205.74 0)
 		(unit 1)
@@
 					(unit 1)
 				)
+			)
+		)
+	)
+	(symbol
+		(lib_id "power:GND")
+		(at 166.37 228.6 0)
+		(unit 1)
+		(body_style 1)
+		(exclude_from_sim no)
+		(in_bom yes)
+		(on_board yes)
+		(in_pos_files yes)
+		(dnp no)
+		(fields_autoplaced yes)
+		(property "Reference" "#PWR024"
+			(at 166.37 234.95 0)
+			(hide yes)
+			(show_name no)
+			(do_not_autoplace no)
+			(effects
+				(font
+					(size 1.27 1.27)
+				)
+			)
+		)
+		(property "Value" "GND"
+			(at 166.37 233.68 0)
+			(show_name no)
+			(do_not_autoplace no)
+			(effects
+				(font
+					(size 1.27 1.27)
+				)
+			)
+		)
+		(property "Footprint" ""
+			(at 166.37 228.6 0)
+			(hide yes)
+			(show_name no)
+			(do_not_autoplace no)
+			(effects
+				(font
+					(size 1.27 1.27)
+				)
+			)
+		)
+		(property "Datasheet" ""
+			(at 166.37 228.6 0)
+			(hide yes)
+			(show_name no)
+			(do_not_autoplace no)
+			(effects
+				(font
+					(size 1.27 1.27)
+				)
+			)
+		)
+		(property "Description" "Power symbol creates a global label with name \"GND\" , ground"
+			(at 166.37 228.6 0)
+			(hide yes)
+			(show_name no)
+			(do_not_autoplace no)
+			(effects
+				(font
+					(size 1.27 1.27)
+				)
+			)
+		)
+		(pin "1"
+		)
+		(instances
+			(project "SolarMeshtasticNodeMini"
+				(path "/256f162e-4f54-42b3-a315-b65231ce36a5"
+					(reference "#PWR024")
+					(unit 1)
+				)

Commit message: pcb, sch: increase RISET from 300Ohm to 360OOhm as it was too close to the short-detect fault detection threshold
Parts:
- R4: value 300 -> 360
Changed lines of the file:
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@@
 			)
 		)
-		(property "Value" "300"
+		(property "Value" "360"
 			(at 48.26 73.6599 0)
 			(show_name no)

Commit message: pcb, sch: add TVS protection to inputs
Parts:
- added D1: SMAJ5.0A, Diode_SMD:D_SMA, symbol Diode:SMAJ5.0A
- added D3: SMAJ15A, Diode_SMD:D_SMA, symbol Diode:SMAJ14A
Connections:
- net GND: now also D1.2 (A2), D3.2 (A2)
- net VBUS: now also D3.1 (A1)
- net VLIPO: now also D1.1 (A1)
Other:
- moved on the sheet: J4

Commit message: pcb, sch: we are using 3V0 everywhere. Also fix misleading comment in schematic regarding SYS voltage within the voltage divier
Connections:
- net +3V3 renamed +3V0
Other:
- note added: "+3V0"
- note added: "SYS is regulated to 4.5V; the 24V concern is input-side only"
- note removed: "+3v3"
- note removed: "Take Care: Solar goes up to 24V! A 1:1 divider will not be enough here."
Changed lines of the file:
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@@
 		)
 	)
-	(text "+3v3"
+	(text "+3V0"
 		(exclude_from_sim no)
 		(at 125.476 21.59 0)
@@
 		)
 	)
-	(text "Take Care: Solar goes \nup to 24V! A 1:1 divider\n will not be enough here."
+	(text "SYS is regulated to 4.5V; \nthe 24V concern is input-side \nonly"
 		(exclude_from_sim no)
-		(at 306.832 51.816 0)
+		(at 307.594 53.848 0)
 		(effects
 			(font
@@
 		)
 	)
-	(label "+3V3"
+	(label "+3V0"
 		(at 295.91 107.95 270)
 		(effects
@@
 		)
 	)
-	(label "+3V3"
+	(label "+3V0"
 		(at 218.44 152.4 0)
 		(effects
@@
 		)
 	)
-	(label "+3V3"
+	(label "+3V0"
 		(at 190.5 97.79 180)
 		(effects
@@
 		)
 	)
-	(label "+3V3"
+	(label "+3V0"
 		(at 118.11 171.45 270)
 		(effects
@@
 		)
 	)
-	(label "+3V3"
+	(label "+3V0"
 		(at 121.92 132.08 180)
 		(effects
@@
 		)
 	)
-	(label "+3V3"
+	(label "+3V0"
 		(at 121.92 139.7 180)
 		(effects
@@
 		)
 	)
-	(label "+3V3"
+	(label "+3V0"
 		(at 214.63 62.23 90)
 		(effects
@@
 		)
 	)
-	(label "+3V3"
+	(label "+3V0"
 		(at 234.95 80.01 0)
 		(effects
@@
 		)
 	)
-	(label "+3V3"
+	(label "+3V0"
 		(at 82.55 182.88 90)
 		(effects
@@
 			)
 		)
-		(property "Value" "+3V3"
+		(property "Value" "+3V0"
 			(at 147.574 25.146 0)
 			(show_name no)

Commit message: pcb, sch: add 1nF C to power switch to limit inrush
Parts:
- added C11: 1nF, Capacitor_SMD:C_0805_2012Metric_Pad1.18x1.45mm_HandSolder, symbol Device:C
Connections:
- net VOUT: now also C11.1
- net at U5.4 (CT): now also C11.2
- no-connect marks 14 -> 13
Changed lines of the file:
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@@
 	)
 	(no_connect
-		(at 194.31 154.94)
-	)
-	(no_connect
 		(at 232.41 74.93)
 	)
@@
 	(wire
 		(pts
+			(xy 180.34 152.4) (xy 180.34 149.86)
+		)
+		(stroke
+			(width 0)
+			(type default)
+		)
+	)
+	(wire
+		(pts
 			(xy 214.63 62.23) (xy 214.63 67.31)
 		)
@@
 	(wire
 		(pts
-			(xy 187.96 152.4) (xy 191.77 152.4)
+			(xy 97.79 86.36) (xy 97.79 92.71)
 		)
 		(stroke
@@
 	(wire
 		(pts
-			(xy 97.79 86.36) (xy 97.79 92.71)
+			(xy 125.73 139.7) (xy 121.92 139.7)
 		)
 		(stroke
@@
 	(wire
 		(pts
-			(xy 125.73 139.7) (xy 121.92 139.7)
+			(xy 78.74 86.36) (xy 82.55 86.36)
 		)
 		(stroke
@@
 	(wire
 		(pts
-			(xy 78.74 86.36) (xy 82.55 86.36)
+			(xy 40.64 133.35) (xy 52.07 133.35)
 		)
 		(stroke
@@
 	(wire
 		(pts
-			(xy 40.64 133.35) (xy 52.07 133.35)
+			(xy 166.37 218.44) (xy 176.53 218.44)
 		)
 		(stroke
@@
 	(wire
 		(pts
-			(xy 166.37 218.44) (xy 176.53 218.44)
+			(xy 83.82 130.81) (xy 83.82 132.08)
 		)
 		(stroke
@@
 	(wire
 		(pts
-			(xy 83.82 130.81) (xy 83.82 132.08)
+			(xy 41.91 76.2) (xy 41.91 80.01)
 		)
 		(stroke
@@
 	(wire
 		(pts
-			(xy 41.91 76.2) (xy 41.91 80.01)
+			(xy 180.34 152.4) (xy 191.77 152.4)
 		)
 		(stroke
@@
 	(wire
 		(pts
+			(xy 180.34 154.94) (xy 194.31 154.94)
+		)
+		(stroke
+			(width 0)
+			(type default)
+		)
+	)
+	(wire
+		(pts
 			(xy 147.32 39.37) (xy 147.32 41.91)
 		)
@@
 	(wire
 		(pts
+			(xy 175.26 157.48) (xy 180.34 157.48)
+		)
+		(stroke
+			(width 0)
+			(type default)
+		)
+	)
+	(wire
+		(pts
 			(xy 41.91 76.2) (xy 45.72 76.2)
 		)
@@
 	(wire
 		(pts
+			(xy 180.34 157.48) (xy 180.34 154.94)
+		)
+		(stroke
+			(width 0)
+			(type default)
+		)
+	)
+	(wire
+		(pts
 			(xy 124.46 222.25) (xy 128.27 222.25)
 		)
@@
 	(wire
 		(pts
+			(xy 180.34 149.86) (xy 175.26 149.86)
+		)
+		(stroke
+			(width 0)
+			(type default)
+		)
+	)
+	(wire
+		(pts
 			(xy 88.9 54.61) (xy 88.9 53.34)
 		)
@@
 					(unit 1)
 				)
+			)
+		)
+	)
+	(symbol
+		(lib_id "Device:C")
+		(at 175.26 153.67 0)
+		(unit 1)
+		(body_style 1)
+		(exclude_from_sim no)
+		(in_bom yes)
+		(on_board yes)
+		(in_pos_files yes)
+		(dnp no)
+		(property "Reference" "C11"
+			(at 171.196 151.638 0)
+			(show_name no)
+			(do_not_autoplace no)
+			(effects
+				(font
+					(size 1.27 1.27)
+				)
+				(justify left)
+			)
+		)
+		(property "Value" "1nF"
+			(at 171.704 155.956 0)
+			(show_name no)
+			(do_not_autoplace no)
+			(effects
+				(font
+					(size 1.27 1.27)
+				)
+				(justify left)
+			)
+		)
+		(property "Footprint" "Capacitor_SMD:C_0805_2012Metric_Pad1.18x1.45mm_HandSolder"
+			(at 176.2252 157.48 0)
+			(hide yes)
+			(show_name no)
+			(do_not_autoplace no)
+			(effects
+				(font
+					(size 1.27 1.27)
+				)
+			)
+		)
+		(property "Datasheet" ""
+			(at 175.26 153.67 0)
+			(hide yes)
+			(show_name no)
+			(do_not_autoplace no)
+			(effects
+				(font
+					(size 1.27 1.27)
+				)
+			)
+		)
+		(property "Description" "Unpolarized capacitor"
+			(at 175.26 153.67 0)
+			(hide yes)
+			(show_name no)
+			(do_not_autoplace no)
+			(effects
+				(font
+					(size 1.27 1.27)
+				)
+			)
+		)
+		(pin "1"
+		)
+		(pin "2"
+		)
+		(instances
+			(project "SolarMeshtasticNodeMini"
+				(path "/256f162e-4f54-42b3-a315-b65231ce36a5"
+					(reference "C11")
+					(unit 1)
+				)

Commit message: pcb, sch: remove tvs from VBat to avoid draining
Parts:
- removed D1: SMAJ5.0A, Diode_SMD:D_SMA, symbol Diode:SMAJ5.0A
- D3: value SMAJ15A -> SMAJ14A
Changed lines of the file:
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@@
 	(text "Battery Connection"
 		(exclude_from_sim no)
-		(at 25.146 154.432 0)
+		(at 25.146 159.512 0)
 		(effects
 			(font
@@
 	)
 	(junction
-		(at 20.32 165.1)
-		(diameter 0)
-		(color 0 0 0 0)
-	)
-	(junction
 		(at 85.09 45.72)
 		(diameter 0)
@@
 	)
 	(junction
-		(at 27.94 165.1)
-		(diameter 0)
-		(color 0 0 0 0)
-	)
-	(junction
 		(at 83.82 130.81)
 		(diameter 0)
@@
 	(wire
 		(pts
-			(xy 20.32 165.1) (xy 22.86 165.1)
+			(xy 19.05 165.1) (xy 22.86 165.1)
 		)
 		(stroke
@@
 	(wire
 		(pts
-			(xy 19.05 165.1) (xy 20.32 165.1)
-		)
-		(stroke
-			(width 0)
-			(type default)
-		)
-	)
-	(wire
-		(pts
 			(xy 166.37 226.06) (xy 166.37 228.6)
 		)
@@
 	(wire
 		(pts
-			(xy 20.32 162.56) (xy 20.32 165.1)
-		)
-		(stroke
-			(width 0)
-			(type default)
-		)
-	)
-	(wire
-		(pts
 			(xy 115.57 80.01) (xy 115.57 85.09)
 		)
@@
 	(wire
 		(pts
-			(xy 25.4 165.1) (xy 27.94 165.1)
-		)
-		(stroke
-			(width 0)
-			(type default)
-		)
-	)
-	(wire
-		(pts
 			(xy 76.2 135.89) (xy 77.47 135.89)
 		)
@@
 	(wire
 		(pts
-			(xy 27.94 165.1) (xy 29.21 165.1)
+			(xy 25.4 165.1) (xy 29.21 165.1)
 		)
 		(stroke
@@
 	(wire
 		(pts
-			(xy 27.94 162.56) (xy 27.94 165.1)
-		)
-		(stroke
-			(width 0)
-			(type default)
-		)
-	)
-	(wire
-		(pts
 			(xy 118.11 166.37) (xy 118.11 171.45)
 		)
@@
 	)
 	(symbol
-		(lib_id "Diode:SMAJ5.0A")
-		(at 24.13 162.56 0)
-		(unit 1)
-		(body_style 1)
-		(exclude_from_sim no)
-		(in_bom yes)
-		(on_board yes)
-		(in_pos_files yes)
-		(dnp no)
-		(fields_autoplaced yes)
-		(property "Reference" "D1"
-			(at 24.13 156.21 0)
-			(show_name no)
-			(do_not_autoplace no)
-			(effects
-				(font
-					(size 1.27 1.27)
-				)
-			)
-		)
-		(property "Value" "SMAJ5.0A"
-			(at 24.13 158.75 0)
-			(show_name no)
-			(do_not_autoplace no)
-			(effects
-				(font
-					(size 1.27 1.27)
-				)
-			)
-		)
-		(property "Footprint" "Diode_SMD:D_SMA"
-			(at 24.13 167.64 0)
-			(hide yes)
-			(show_name no)
-			(do_not_autoplace no)
-			(effects
-				(font
-					(size 1.27 1.27)
-				)
-			)
-		)
-		(property "Datasheet" "https://www.littelfuse.com/media?resourcetype=datasheets&itemid=75e32973-b177-4ee3-a0ff-cedaf1abdb93&filename=smaj-datasheet"
-			(at 22.86 162.56 0)
-			(hide yes)
-			(show_name no)
-			(do_not_autoplace no)
-			(effects
-				(font
-					(size 1.27 1.27)
-				)
-			)
-		)
-		(property "Description" "400W unidirectional Transient Voltage Suppressor, 5.0Vr, SMA(DO-214AC)"
-			(at 24.13 162.56 0)
-			(hide yes)
-			(show_name no)
-			(do_not_autoplace no)
-			(effects
-				(font
-					(size 1.27 1.27)
-				)
-			)
-		)
-		(pin "1"
-		)
-		(pin "2"
-		)
-		(instances
-			(project "SolarMeshtasticNodeMini"
-				(path "/256f162e-4f54-42b3-a315-b65231ce36a5"
-					(reference "D1")
-					(unit 1)
-				)
-			)
-		)
-	)
-	(symbol
 		(lib_id "power:+3V0")
 		(at 147.32 29.21 0)
@@
 			)
 		)
-		(property "Value" "SMAJ15A"
+		(property "Value" "SMAJ14A"
 			(at 24.13 129.54 0)
 			(show_name no)

Commit message: pcb, sch: GPIO is the NSS of the SX1262. Do not pull high.
Connections:
- net +3V0: no longer U2.16 (GPIO8)
- no-connect marks 13 -> 14
Changed lines of the file:
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@@
+	)
+	(no_connect
+		(at 232.41 80.01)
 	)
 	(no_connect
@@
 	(wire
 		(pts
-			(xy 232.41 80.01) (xy 234.95 80.01)
-		)
-		(stroke
-			(width 0)
-			(type default)
-		)
-	)
-	(wire
-		(pts
 			(xy 78.74 45.72) (xy 85.09 45.72)
 		)
@@
 		(effects
 			(font
-				(size 1.27 1.27)
-			)
-			(justify left bottom)
-		)
-	)
-	(label "+3V0"
-		(at 234.95 80.01 0)
-		(effects
-			(font
